File: NanoFreak.kicad_pcb (KiCad board)
At the start: 4 copper layers, 233.5 x 118.5 mm, 99 parts, among them J1 Audio Out, J2 MIDI In, J3 Micro_SD_Card, SW1 Control Rotary, SW10 Key 6, SW11 Key 7, SW12 Key 8, SW13 Key 9, SW14 Key 10, SW15 Key 11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

Commit message: Add files via upload
Connections:
- J2 pad R: Net-(J2-PadR) -> Net-(D4-A)
- J2 pad S: Net-(D4-A) -> unconnected-(J2-PadS)
- J2 pad T: unconnected-(J2-PadT) -> Net-(J2-PadT)
- R18 pad 1: +3.3V -> +3V3
- R19 pad 1: Net-(J2-PadR) -> Net-(J2-PadT)
- R20 pad 1: +3.3V -> +3V3
- R22 pad 1: +3.3V -> +3V3
- U4 pad 8: +3.3V -> +3V3
Routing:
- net Net-(J2-PadR): track 13.9 -> 0.00 mm
- net Net-(D4-A): track 13.1 -> 18.4 mm
- net Net-(J2-PadT): track 0.00 -> 4.10 mm
- net unconnected-(J2-PadS): track 0.00 -> 0.50 mm
Changed lines of the file:
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@@
 	(net 39 "Net-(U3-PROG3)")
 	(net 40 "Net-(U3-CE)")
-	(net 41 "Net-(J2-PadR)")
+	(net 41 "Net-(J2-PadT)")
 	(net 42 "Net-(D4-K)")
 	(net 43 "Net-(U4-VO1)")
@@
 	(net 94 "Net-(U5-INTA)")
 	(net 95 "Net-(D4-A)")
-	(net 96 "unconnected-(J2-PadT)")
+	(net 96 "unconnected-(J2-PadS)")
 	(net 97 "unconnected-(U4-NC-Pad4)")
 	(net 98 "unconnected-(U4-NC-Pad1)")
 	(net 99 "Net-(U2-XSMT)")
 	(net 100 "Net-(U2-LDOO)")
+	(net 101 "+3V3")
 	(footprint "Resistor_SMD:R_0603_1608Metric"
 		(layer "F.Cu")
@@
 			(layers "F.Cu" "F.Mask" "F.Paste")
 			(roundrect_rratio 0.25)
-			(net 13 "+3.3V")
+			(net 101 "+3V3")
 			(pintype "passive")
 		)
@@
 			(layers "F.Cu" "F.Mask" "F.Paste")
 			(roundrect_rratio 0.25)
-			(net 13 "+3.3V")
+			(net 101 "+3V3")
 			(pintype "passive")
 		)
@@
 			(layers "F.Cu" "F.Mask" "F.Paste")
 			(roundrect_rratio 0.25)
-			(net 41 "Net-(J2-PadR)")
+			(net 41 "Net-(J2-PadT)")
 			(pintype "passive")
 		)
@@
 			(layers "F.Cu" "F.Mask" "F.Paste")
 			(roundrect_rratio 0.25)
-			(net 13 "+3.3V")
+			(net 101 "+3V3")
 			(pintype "passive")
 		)
@@
 			(layers "*.Cu" "*.Mask")
 			(remove_unused_layers no)
-			(net 41 "Net-(J2-PadR)")
+			(net 95 "Net-(D4-A)")
 			(pintype "passive")
 		)
@@
 			(layers "*.Cu" "*.Mask")
 			(remove_unused_layers no)
-			(net 95 "Net-(D4-A)")
+			(net 96 "unconnected-(J2-PadS)")
 			(pintype "passive")
 		)
@@
 			(layers "*.Cu" "*.Mask")
 			(remove_unused_layers no)
-			(net 96 "unconnected-(J2-PadT)")
+			(net 41 "Net-(J2-PadT)")
 			(pintype "passive")
 		)
@@
 			(layers "*.Cu" "*.Mask")
 			(remove_unused_layers no)
-			(net 13 "+3.3V")
+			(net 101 "+3V3")
 			(pinfunction "VCC")
 			(pintype "passive")
@@
 	)
 	(segment
-		(start 146.35 33.15)
-		(end 148.5 31)
+		(start 135.85 33.15)
+		(end 138.5 30.5)
 		(width 0.2)
 		(layer "F.Cu")
@@
 	(segment
 		(start 135.5 33.15)
-		(end 146.35 33.15)
+		(end 135.85 33.15)
 		(width 0.2)
 		(layer "F.Cu")
@@
 	)
 	(segment
-		(start 141 28)
-		(end 143 26)
-		(width 0.2)
-		(layer "F.Cu")
-		(net 95)
-	)
-	(segment
-		(start 136.5 27.25)
-		(end 137.25 28)
+		(start 131.5 27.23)
+		(end 135.48 27.23)
 		(width 0.2)
 		(layer "F.Cu")
@@
 	)
 	(segment
-		(start 137.25 28)
-		(end 141 28)
+		(start 145.25 27.25)
+		(end 136.5 27.25)
 		(width 0.2)
 		(layer "F.Cu")
@@
 	)
 	(segment
-		(start 131.5 27.23)
-		(end 135.48 27.23)
+		(start 135.48 27.23)
+		(end 135.5 27.25)
 		(width 0.2)
 		(layer "F.Cu")
@@
 	)
 	(segment
-		(start 135.48 27.23)
-		(end 135.5 27.25)
+		(start 148.5 30.5)
+		(end 145.25 27.25)
 		(width 0.2)
 		(layer "F.Cu")
@@
 		(width 0.2)
 		(layer "F.Cu")
-		(net 95)
+		(net 96)
 	)
 	(segment

Commit message: Add files via upload
Parts:
- removed C16, C17: 0.1µf, Capacitor_SMD:C_0603_1608Metric_Pad1.08x0.95mm_HandSolder
- added SW18: SW_SPDT, Button_Switch_SMD:SW_SPDT_PCM12, F.Cu at (38.1, 23.5)
- R12, R28, R29: value 220 -> 10k
- RV1, RV2, RV3, RV4, RV5, RV6, RV7: footprint Potentiometer_THT:Potentiometer_Vishay_248GJ-249GJ_Single_Vertical -> PotentiometerTHT:Potentiometer
- SW10: value Key 6 -> Key 7
- SW11: value Key 7 -> Key 2
- SW12: value Key 8 -> Key 1
- SW13: value Key 9 -> Key 4
- SW14: value Key 10 -> Key 3
- SW15: value Key 11 -> Key 6
- SW16: value Key 12 -> Key 5
- SW5: value Key 1 -> Key 10
- SW6: value Key 2 -> Key 12
- SW7: value Key 3 -> Key 9
- SW8: value Key 4 -> Key 11
- SW9: value Key 5 -> Key 8
- moved SW5 15.0 mm to (94.3, 120.9)
- moved SW6 12.0 mm to (104.0, 100.4)
- moved SW7 12.0 mm to (116.8, 120.9)
- moved SW8 9.00 mm to (126.5, 100.4)
- moved SW9 9.00 mm to (139.3, 120.9)
- moved C1 8.45 mm to (139.2, 85.6)
- moved C2 8.45 mm to (156.7, 85.1)
- moved R1 8.45 mm to (139.2, 79.6)
- moved R2 8.45 mm to (139.2, 81.1)
- moved R3 8.45 mm to (139.2, 82.6)
- moved R4 8.45 mm to (139.2, 84.1)
- moved R5 8.45 mm to (156.7, 80.6)
- moved R6 8.45 mm to (156.7, 82.6)
- moved U5 8.45 mm to (147.9, 88.1)
- moved U1 7.06 mm to (70.5, 76.8)
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Connections:
- R18 pad 1: +3V3 -> +3.3V
- R20 pad 1: +3V3 -> +3.3V
- R22 pad 1: +3V3 -> +3.3V
- SW10 pad 1: Net-(U5-GPB5) -> Net-(U5-GPA0)
- SW11 pad 1: Net-(U5-GPA0) -> Net-(U5-GPB1)
- SW12 pad 1: Net-(U5-GPA1) -> Net-(U5-GPB0)
- SW13 pad 1: Net-(U5-GPA2) -> Net-(U5-GPB3)
- SW14 pad 1: Net-(U5-GPA3) -> Net-(U5-GPB2)
- SW15 pad 1: Net-(U5-GPA4) -> Net-(U5-GPB5)
- SW16 pad 1: Net-(U5-GPA5) -> Net-(U5-GPB4)
- SW5 pad 1: Net-(U5-GPB0) -> Net-(U5-GPA3)
- SW6 pad 1: Net-(U5-GPB1) -> Net-(U5-GPA5)
- SW7 pad 1: Net-(U5-GPB2) -> Net-(U5-GPA2)
- SW8 pad 1: Net-(U5-GPB3) -> Net-(U5-GPA4)
- SW9 pad 1: Net-(U5-GPB4) -> Net-(U5-GPA1)
- U3 pad 14: Net-(BT1-+) -> Net-(SW18-A)
- U3 pad 15: Net-(BT1-+) -> Net-(SW18-A)
- U3 pad 16: Net-(BT1-+) -> Net-(SW18-A)
- U4 pad 8: +3V3 -> +3.3V
Routing:
- net +3.3V: track 584.3 -> 44.5 mm, vias 9 -> 13
- net Net-(BT1-+): track 76.4 -> 5.65 mm
- net Net-(SW18-A): track 0.00 -> 68.1 mm
- net Net-(U5-GPA5): track 109.3 -> 47.9 mm
- net Net-(U5-GPA4): track 88.6 -> 27.7 mm
- net GND: track 118.8 -> 76.0 mm, vias 30 -> 36
- net Net-(U5-GPB1): track 55.3 -> 21.2 mm, vias 1 -> 0
- net STICKX: track 59.1 -> 92.9 mm
- net Net-(U5-GPA1): track 71.3 -> 38.2 mm
- net Net-(U5-GPB0): track 75.9 -> 43.4 mm, vias 1 -> 0
- net +5V: track 43.1 -> 12.3 mm, vias 2 -> 4
- net Net-(U5-GPA2): track 83.9 -> 55.8 mm, vias 2 -> 0
- net Net-(U5-GPB3): track 66.1 -> 44.8 mm
- net Net-(U5-GPB4): track 68.5 -> 89.0 mm
- net Net-(U5-GPA3): track 92.9 -> 76.2 mm
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- added copper zone on In2.Cu, net +3.3V
- added copper zone on In2.Cu, net +5V
- removed copper zone on F.Cu, net GND
