File: NanoFreak.kicad_sch (KiCad schematic)
At the start: 92 parts, among them J1 Audio Out, J2 MIDI In, J3 Micro_SD_Card, SW1 Control Rotary, SW10 Key 6, SW11 Key 7, SW12 Key 8, SW13 Key 9, SW14 Key 10, SW15 Key 11, SW16 Key 12, SW17 Filter Type, SW2 Oct +, SW3 Shift Key, SW4 Oct -, SW5 Key 1, SW6 Key 2, SW7 Key 3, SW8 Key 4, SW9 Key 5, U1 ESP32-S3-DevKitC, U2 PCM5102A, U3 MCP73871, U4 6N138, U5 MCP23017_SO, U6 MCP1700T-3302E/MB, U7 THB001P, U8 OLED

Commit message: Add files via upload
Connections:
- net at D4.2 (A), U4.3 (C2): now also J2.R; no longer J2.S
- net at R19.1: now also J2.T; no longer J2.R
Other:
- moved on the sheet: J2
Changed lines of the file:
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@@
 	(wire
 		(pts
+			(xy 40.64 203.2) (xy 40.64 213.36)
+		)
+		(stroke
+			(width 0)
+			(type default)
+		)
+	)
+	(wire
+		(pts
 			(xy 334.01 232.41) (xy 314.96 232.41)
 		)
@@
 	(wire
 		(pts
-			(xy 40.64 203.2) (xy 40.64 213.36)
-		)
-		(stroke
-			(width 0)
-			(type default)
-		)
-	)
-	(wire
-		(pts
 			(xy 363.22 184.15) (xy 363.22 190.5)
 		)
@@
 	(wire
 		(pts
-			(xy 39.37 205.74) (xy 41.91 205.74)
-		)
-		(stroke
-			(width 0)
-			(type default)
-		)
-	)
-	(wire
-		(pts
 			(xy 330.2 204.47) (xy 332.74 204.47)
 		)
@@
 	(wire
 		(pts
+			(xy 40.64 203.2) (xy 39.37 203.2)
+		)
+		(stroke
+			(width 0)
+			(type default)
+		)
+	)
+	(wire
+		(pts
 			(xy 382.27 95.25) (xy 382.27 104.14)
 		)
@@
 	(wire
 		(pts
+			(xy 41.91 205.74) (xy 39.37 205.74)
+		)
+		(stroke
+			(width 0)
+			(type default)
+		)
+	)
+	(wire
+		(pts
 			(xy 332.74 217.17) (xy 330.2 217.17)
 		)
@@
 	(wire
 		(pts
-			(xy 39.37 203.2) (xy 40.64 203.2)
-		)
-		(stroke
-			(width 0)
-			(type default)
-		)
-	)
-	(wire
-		(pts
 			(xy 57.15 151.13) (xy 53.34 151.13)
 		)
@@
 	(symbol
 		(lib_id "Connector_Audio:AudioJack3")
-		(at 34.29 205.74 0)
+		(at 34.29 203.2 0)
 		(unit 1)
 		(exclude_from_sim no)
@@
 		(fields_autoplaced yes)
 		(property "Reference" "J2"
-			(at 32.385 196.85 0)
+			(at 32.385 194.31 0)
 			(effects
 				(font
@@
 		)
 		(property "Value" "MIDI In"
-			(at 32.385 199.39 0)
+			(at 32.385 196.85 0)
 			(effects
 				(font
@@
 		)
 		(property "Footprint" "Connector_Audio:Jack_3.5mm_CUI_SJ1-3523N_Horizontal"
-			(at 34.29 205.74 0)
+			(at 34.29 203.2 0)
 			(effects
 				(font
@@
 		)
 		(property "Datasheet" "~"
-			(at 34.29 205.74 0)
+			(at 34.29 203.2 0)
 			(effects
 				(font
@@
 		)
 		(property "Description" "Audio Jack, 3 Poles (Stereo / TRS)"
-			(at 34.29 205.74 0)
+			(at 34.29 203.2 0)
 			(effects
 				(font

Commit message: Add files via upload
Parts:
- removed C16, C17: 0.1µf, Capacitor_SMD:C_0603_1608Metric_Pad1.08x0.95mm_HandSolder, symbol Device:C
- added SW18: SW_SPDT, Button_Switch_SMD:SW_SPDT_PCM12, symbol Switch:SW_SPDT
- R12, R28, R29: value 220 -> 10k
- RV1, RV2, RV3, RV4, RV5, RV6, RV7: footprint Potentiometer_THT:Potentiometer_Vishay_248GJ-249GJ_Single_Vertical -> PotentiometerTHT:Potentiometer
- renumbered SW11 to SW10, SW6 to SW11, SW5 to SW12, SW8 to SW13, SW7 to SW14, SW10 to SW15, SW9 to SW16, SW14 to SW5, SW16 to SW6, SW13 to SW7, SW15 to SW8, SW12 to SW9
Connections:
- net +3V3 is gone; now on net +3.3V: R18.1, R20.1, R22.1, U4.8 (VCC)
- net at U3.14 (V_{BAT}), U3.15 (V_{BAT}), U3.16 (V_{BAT_SENSE}): now also SW18.1 (A); no longer BT1.1 (+), C11.1
- new net: BT1.1 (+), C11.1, SW18.2 (B)
Other:
- moved on the sheet: BT1, C11
